Commit message: heightfield export

File: resources/robots/a1/urdf/a1_obj.urdf (robot description, URDF)
Before this commit: robot a1_description, 21 links, 20 joints
Links:
- link FL_calf: geometry collision box size=0.2 0.016 0.016
- link FL_hip: geometry 
- link FL_thigh: geometry collision box size=0.2 0.0245 0.034
- link FR_calf: geometry collision box size=0.2 0.016 0.016
- link FR_hip: geometry 
- link FR_thigh: geometry collision box size=0.2 0.0245 0.034
- link RL_calf: geometry 
- link RL_hip: geometry 
- link RL_thigh: geometry collision box size=0.2 0.0245 0.034
- link RR_calf: geometry collision box size=0.2 0.016 0.016
- link RR_hip: geometry 
- link RR_thigh: geometry collision box size=0.2 0.0245 0.034
